File: Devboard/Devboard.kicad_sch (KiCad schematic)
At the start: 23 parts, among them IC1 114993390, SW1 SHPHLD, U1 E73-2G4M08S1C, U2 NPM1300-QEAA-R7, Y1 32.768

Commit message: Continued design
Parts:
- removed C1, C2: 22p, symbol Device:C
- removed C3: 1u, symbol Device:C
- removed IC1: 114993390, Project_Components:114993390, symbol Project_Components:114993390
- removed L1: 2u2, symbol Device:L_Small
- removed R2: 150k, symbol Device:R
- removed R3: 47k, symbol Device:R
- removed SW1: SHPHLD, symbol Switch:SW_Push
- removed U1: E73-2G4M08S1C, E73-2G4M08S1C:E73-2G4M08S1C, symbol E73-2G4M08S1C:E73-2G4M08S1C
- removed U2: NPM1300-QEAA-R7, QFN32_5X5_NOR, symbol 2026-05-19_19-41-51:NPM1300-QEAA-R7
- added C19: 10u, symbol Device:C
- added C20, C21: 1u, symbol Device:C
- added C22: 2u2, symbol Device:C
- added FB1: LI0603G121R-10, Inductor_SMD:L_1206_3216Metric_Pad1.22x1.90mm_HandSolder, symbol Device:FerriteBead
- added IC2: 114993390, Project_Components:114993390, symbol Project_Components:114993390
- added J8: USB_C_Receptacle_USB2.0_16P, Connector_USB:USB_C_Receptacle_GCT_USB4105-xx-A_16P_TopMnt_Horizontal, symbol Connector:USB_C_Receptacle_USB2.0_16P
- added L4: 10u(DNP), symbol Device:L_Small
- added L5, L6: 2u2, symbol Device:L_Small
- added R10: 47k, symbol Device:R
- added R6, R7, R8: R_Small, symbol Device:R_Small
- added R9: 150k, symbol Device:R
- added SW3: SW_Push, symbol Switch:SW_Push
- added SW4: SHPHLD, symbol Switch:SW_Push
- added U12: SRV05-4, Package_TO_SOT_SMD:SOT-23-6_Handsoldering, symbol Power_Protection:SRV05-4
- added U2: E73-2G4M08S1C, E73-2G4M08S1C:E73-2G4M08S1C, symbol E73-2G4M08S1C:E73-2G4M08S1C
- added U4: NPM1300-QEAA-R7, QFN32_5X5_NOR, symbol 2026-05-19_19-41-51:NPM1300-QEAA-R7
- C4: value 10u -> 22p
- C6: value 100n -> 22p
- C7: value 1u -> 10u
- C8: value 2u2 -> 10u
- C9: value 10u -> 100n
Connections:
- net CC1: now also J8.A5 (CC1), U4.24 (CC2)
- net CC2: now also J8.B5 (CC2), U4.23 (CC1)
- net GND: now also C4.1, C6.1, C9.2, C19.1, C20.1, C21.1, C22.1, IC2.10 (GND_2), IC2.7 (GND_1), J8.A1 (GND), J8.A12 (GND), J8.B1 (GND), J8.B12 (GND), J8.S1 (SHIELD), R10.2, R9.2, SW3.2, SW4.2, U12.2 (VN), U2.21 (GND@2), U2.24 (GND@3), U2.5 (GND@1), U4.33 (AVSS); no longer C11.1, C6.2, C7.1, C8.1
- net NTC: now also U4.18 (NTC)
- net PVSS1: now also C10.1, C8.1, U4.2 (PVSS1); no longer C4.1, C9.1
- net PVSS2: now also C11.1, C7.2, U4.6 (PVSS2); no longer C10.1
- net SCL: now also U2.7 (P0.02/AIN0), U4.14 (SCL)
- net SDA: now also U2.3 (P0.03/AIN1), U4.13 (SDA)
- net SW2: now also L5.2, U4.5 (SW2)
- net VBAT: now also C22.2, U4.19 (VBAT); no longer C8.2
- net VBUS: now also C21.2, FB1.1, FB1.2, J8.A4 (VBUS), J8.A9 (VBUS), J8.B4 (VBUS), J8.B9 (VBUS), U4.21 (VBUS); no longer C7.2
- net VBUSOUT: now also C20.2, U2.27 (VBUS), U4.22 (VBUSOUT)
- net VSYS: now also C19.2, R6.2, R7.2, R8.2, U4.20 (VSYS), U4.28 (LSIN1/VINLDO1), U4.4 (PVDD); no longer C9.2
- net at D3.1 (K): now also U4.25 (LED0)
- net at D2.1 (K): now also U4.26 (LED1)
- net at D1.1 (K): now also U4.27 (LED2)
- net at D3.2 (A): now also R8.1
- net at D1.2 (A): now also R6.1
- net at Y1.1: now also C6.2, U2.13 (P0.01/XL2)
- net at Y1.2: now also C4.2, U2.11 (P0.00/XL1)
- net at D2.2 (A): now also R7.1
- removed net +1V8: C4.2, C6.1
- new net: L4.1, U2.25 (DCCH)
- new net: SW3.1, U2.26 (P0.18/RESET)
- new net: R9.1, U4.16 (VSET2)
- new net: C7.1, L5.1, U4.30 (LSIN2/VINLDO2), U4.32 (VOUT2)
- new net: SW4.1, U4.15 (SHPHLD)
- new net: R10.1, U4.17 (VSET1)
- new net: L6.1, U4.3 (SW1)
- new net +3.3V: IC2.8 (VCC), U4.31 (LSOUT2/VOUTLDO2)
- new net +5V: U12.5 (VP)
- new net BM_INT: U2.15 (P0.05/AIN3), U4.8 (GPIO1)
- new net BM_RST: U2.18 (P0.04/AIN2), U4.7 (GPIO0)
- new net D+: J8.A6 (D+), J8.B6 (D+), U12.1 (IO1), U2.29 (DM)
- new net D-: J8.A7 (D-), J8.B7 (D-), U12.6 (IO4), U2.31 (DP)
- new net LoRa_BUSY: IC2.11 (BUSY), U2.1 (P1.11)
- new net LoRa_MISO: IC2.2 (MISO), U2.38 (P1.02)
- new net LoRa_MOSI: IC2.3 (MOSI), U2.40 (P1.04)
- new net LoRa_NSS: IC2.6 (NSS), U2.2 (P1.10)
- new net LoRa_RST: IC2.5 (NRST), U2.17 (P1.09)
- new net LoRa_SCK: IC2.4 (SCK), U2.42 (P1.06)
- new net LoRa_SW: IC2.1 (RF_SW_), U2.36 (P1.00)
- new net SWDCLK: U2.39 (SWDCLK)
- new net SWDIO: U2.37 (SWDIO)
- new net VLDO: U4.29 (LSOUT1/VOUTLDO1)
- new net VMCU: C8.2, C9.1, L4.2, L6.2, U2.19 (VDD), U2.23 (VDDH), U4.1 (VOUT1), U4.12 (VDDIO)
- no-connect marks 5 -> 9

Commit message: Finished design and layout
Parts:
- removed R7, R8: R_Small, symbol Device:R_Small
- removed U2: E73-2G4M08S1C, E73-2G4M08S1C:E73-2G4M08S1C, symbol E73-2G4M08S1C:E73-2G4M08S1C
- added J2: SWD, Connector_PinHeader_2.54mm:PinHeader_2x03_P2.54mm_Vertical, symbol Connector_Generic:Conn_02x03_Odd_Even
- added J3: RMF, Connector_PinHeader_2.54mm:PinHeader_1x02_P2.54mm_Vertical, symbol Connector:Conn_01x02_Pin
- added R4, R5: 300, Resistor_SMD:R_1206_3216Metric_Pad1.30x1.75mm_HandSolder, symbol Device:R_Small
- added SW3: SW_Push, Button_Switch_SMD:SW_Push_1P1T_NO_CK_KMR2, symbol Switch:SW_Push
- added U2: E73-2G4M08S1C, Project_Components:E73-2G4M08S1C, symbol Project_Components:E73-2G4M08S1C
- C1: renamed from C8; footprint (none) -> Capacitor_SMD:C_1206_3216Metric_Pad1.33x1.80mm_HandSolder
- C10: renamed from C4; footprint (none) -> Capacitor_SMD:C_1206_3216Metric_Pad1.33x1.80mm_HandSolder
- C11: renamed from C6; footprint (none) -> Capacitor_SMD:C_1206_3216Metric_Pad1.33x1.80mm_HandSolder
- C2: renamed from C9; footprint (none) -> Capacitor_SMD:C_1206_3216Metric_Pad1.33x1.80mm_HandSolder
- C3: renamed from C20; footprint (none) -> Capacitor_SMD:C_1206_3216Metric_Pad1.33x1.80mm_HandSolder
- C4: renamed from C7; footprint (none) -> Capacitor_SMD:C_1206_3216Metric_Pad1.33x1.80mm_HandSolder
- C5: renamed from C10; footprint (none) -> Capacitor_SMD:C_1206_3216Metric_Pad1.33x1.80mm_HandSolder
- C6: renamed from C21; footprint (none) -> Capacitor_SMD:C_1206_3216Metric_Pad1.33x1.80mm_HandSolder
- C7: renamed from C22; footprint (none) -> Capacitor_SMD:C_1206_3216Metric_Pad1.33x1.80mm_HandSolder
- C8: renamed from C11; footprint (none) -> Capacitor_SMD:C_1206_3216Metric_Pad1.33x1.80mm_HandSolder
- C9: renamed from C19; footprint (none) -> Capacitor_SMD:C_1206_3216Metric_Pad1.33x1.80mm_HandSolder
- D1, D2, D3: value LED_Small -> Amber; footprint (none) -> LED_SMD:LED_1206_3216Metric_Pad1.42x1.75mm_HandSolder
- L1: renamed from L6; footprint (none) -> Inductor_SMD:L_0805_2012Metric_Pad1.05x1.20mm_HandSolder
- L2: renamed from L5; footprint (none) -> Inductor_SMD:L_0805_2012Metric_Pad1.05x1.20mm_HandSolder
- L3: renamed from L4; footprint (none) -> Inductor_SMD:L_Changjiang_FTC201610D
- R1: renamed from R9; footprint (none) -> Resistor_SMD:R_1206_3216Metric_Pad1.30x1.75mm_HandSolder
- R2: renamed from R10; footprint (none) -> Resistor_SMD:R_1206_3216Metric_Pad1.30x1.75mm_HandSolder
- R3: renamed from R6; value R_Small -> 300; footprint (none) -> Resistor_SMD:R_1206_3216Metric_Pad1.30x1.75mm_HandSolder
- SW1: renamed from SW4; footprint (none) -> Button_Switch_SMD:SW_Push_1P1T_NO_CK_KMR2
- SW2: renamed from SW3; value SW_Push -> RST; footprint (none) -> Button_Switch_SMD:SW_Push_1P1T_NO_CK_KMR2
- U1: renamed from U4; value NPM1300-QEAA-R7 -> NPM1304-QEAA-R; footprint QFN32_5X5_NOR -> Project_Components:QFN32_5X5_NOR
- Y1: footprint (none) -> Crystal:Crystal_SMD_MicroCrystal_CC1V-T1A-2Pin_8.0x3.7mm
- renumbered IC2 to IC1, J8 to J1, U12 to U3
Connections:
- net BM_INT: now also U2.15 (P0.05/AIN3)
- net BM_RST: now also U2.18 (P0.04/AIN2)
- net D+: now also U2.31 (DP)
- net D-: now also U2.29 (DM)
- net GND: now also J2.5 (Pin_5), J3.2 (Pin_2), SW3.2, U2.21 (GND@2), U2.24 (GND@3), U2.5 (GND@1)
- net LoRa_BUSY: now also U2.1 (P1.11)
- net LoRa_MISO: now also U2.38 (P1.02)
- net LoRa_MOSI: now also U2.40 (P1.04)
- net LoRa_NSS: now also U2.2 (P1.10)
- net LoRa_RST: now also U2.17 (P1.09)
- net LoRa_SCK: now also U2.42 (P1.06)
- net LoRa_SW: now also U2.36 (P1.00)
- net SCL: now also U2.4 (P0.28/AIN4)
- net SDA: now also U2.3 (P0.03/AIN1)
- net SWDCLK: now also J2.4 (Pin_4), U2.39 (SWDCLK)
- net SWDIO: now also J2.2 (Pin_2), U2.37 (SWDIO)
- net VBUS: no longer FB1.1, J1.A4 (VBUS), J1.A9 (VBUS), J1.B4 (VBUS), J1.B9 (VBUS)
- net VBUSOUT: now also U2.27 (VBUS)
- net VMCU: now also U2.19 (VDD), U2.23 (VDDH)
- net VSYS: now also R4.2, R5.2
- net at L3.1: now also U2.25 (DCCH)
- net RST: now reaches SW2.1
- net RST: now also J2.3 (Pin_3), U2.26 (P0.18/RESET)
- net at D2.2 (A): now also R4.1
- net at C11.2, Y1.1: now also U2.13 (P0.01/XL2)
- net at C10.2, Y1.2: now also U2.11 (P0.00/XL1)
- net at D3.2 (A): now also R5.1
- new net: FB1.1, J1.A4 (VBUS), J1.A9 (VBUS), J1.B4 (VBUS), J1.B9 (VBUS)
- new net +3V3: J2.1 (Pin_1)
- new net RMF: J3.1 (Pin_1), U2.10 (P0.30/AIN6)
- new net SW0: SW3.1, U2.9 (P0.31/AIN7)
- no-connect marks 9 -> 26
Other:
- moved on the sheet: IC1, SW2
